File: altbier-proto/AltbierProto.kicad_pcb (KiCad board)
At the start: 2 copper layers, 76.2 x 82.5 mm, 103 parts

Commit message: initial commit
Parts:
- added G***: LOGO, kml-custom:FAST-Logo-Medium, F.Cu at (140.6, 76.7)
- added Ref**: Val**, kml-custom:OSHW_Logo_8mm, B.Cu at (141.2, 61.9)
- Battery: renamed from REF**; footprint 0_local:PinHeader_1x02_P2.54mm_Vertical -> Connector_PinHeader_2.54mm:PinHeader_1x02_P2.54mm_Vertical
- G***: footprint 0_alt_bier:logo-alt_bier-1100dpi-8x21mm-front -> altbier:logo-alt_bier-1100dpi-8x21mm-front; moved to B.Cu
- REF** (x24): value Proto_A_Pins_P2.54mm -> Proto_A_Pins_2_P2.54mm; footprint 0_local:Proto_A_Pins_P2.54mm -> Proto:Proto_A_Pins_2_P2.54mm
- REF** (x54): footprint 0_local:Proto_B_Pins_P2.54mm -> Proto:Proto_B_Pins_P2.54mm
- REF** (x2): footprint 0_local:Proto_C_Pins_2x30_P2.54mm -> Proto:Proto_C_Pins_2x30_P2.54mm
- REF** (x6): footprint 0_local:Proto_1206_Pads_1.42x1.75mm_HandSolder -> Proto:Proto_1206_Pads_1.42x1.75mm_HandSolder
- REF** (x6): footprint 0_local:Proto_0805_Pads_1.15x1.40mm_HandSolder -> Proto:Proto_0805_Pads_1.15x1.40mm_HandSolder
- REF** (x6): footprint 0_local:Proto_0603_Pads_1.05x0.95mm_HandSolder -> Proto:Proto_0603_Pads_1.05x0.95mm_HandSolder
- SOP16: value IC_SOIC-16_3.9x9.9mm_Pitch1.27mm -> SOIC-16_3.9x9.9mm_P1.27mm; footprint 0_local:IC_SOIC-16_3.9x9.9mm_Pitch1.27mm -> Package_SO:SOIC-16_3.9x9.9mm_P1.27mm
- TSSOP20: value IC_TSSOP-20_4.4x6.5mm_P0.65mm_thin -> TSSOP-20_4.4x6.5mm_P0.65mm; footprint 0_local:IC_TSSOP-20_4.4x6.5mm_P0.65mm_thin -> Package_SO:TSSOP-20_4.4x6.5mm_P0.65mm
- USB: footprint 0_local:Proto_USB_Micro-B_Jing -> Proto:Proto_USB_Micro-B_Jing
- moved G*** 0.13 mm to (141.1, 104.9)
Other:
- board text added: "Altbier's Proto PCB Rev 02"
- board text added: "Cam's Rev Altbier's Proto PCB"
- board text added: "Micro-B"
- board text removed: "Altbier's Proto PCB Rev 01"
- board text removed: "Battery"
