File: protoplus/protoplus.kicad_pcb (KiCad board)
At the start: 2 copper layers, 24.4 x 32.7 mm, 108 parts

Commit message: initial commit
Parts:
- added REF**: MountingHole_2.2mm_M2, MountingHole:MountingHole_2.2mm_M2, F.Cu at (145.8, 90.7)
- added REF**: protoplus_perfdot, Proto:protoplus_perfdot, F.Cu at (154.9, 55.8)
- added REF**: protoplus_perfdot, Proto:protoplus_perfdot, F.Cu at (160.0, 55.8)
- added REF**: protoplus_perfdot, Proto:protoplus_perfdot, F.Cu at (154.9, 88.8)
- added REF**: protoplus_perfdot, Proto:protoplus_perfdot, F.Cu at (152.4, 88.8)
- added REF**: protoplus_perfdot, Proto:protoplus_perfdot, F.Cu at (152.4, 55.8)
- added REF**: protoplus_perfdot, Proto:protoplus_perfdot, F.Cu at (157.4, 55.8)
- added REF**: protoplus_perfdot, Proto:protoplus_perfdot, F.Cu at (160.0, 88.8)
- added REF**: MountingHole_2.2mm_M2, MountingHole:MountingHole_2.2mm_M2, F.Cu at (164.7, 90.7)
- added REF**: protoplus_perfdot, Proto:protoplus_perfdot, F.Cu at (149.8, 88.8)
- added REF**: MountingHole_2.2mm_M2, MountingHole:MountingHole_2.2mm_M2, F.Cu at (145.8, 53.8)
- added REF**: MountingHole_2.2mm_M2, MountingHole:MountingHole_2.2mm_M2, F.Cu at (164.7, 53.8)
- added REF**: protoplus_perfdot, Proto:protoplus_perfdot, F.Cu at (149.8, 55.8)
- added REF**: protoplus_perfdot, Proto:protoplus_perfdot, F.Cu at (157.4, 88.8)
- added Ref**: Val**, kml-custom:OSHW_Logo_4mm, F.Cu at (157.4, 91.6)
- REF** (x108): value Perfdot -> protoplus_perfdot; footprint Perfboard:Perfdot -> Proto:protoplus_perfdot
- moved REF** 0.13 mm to (160.0, 86.2)
- moved REF** 0.13 mm to (149.8, 58.3)
- moved REF** 0.13 mm to (149.8, 76.1)
- moved REF** 0.13 mm to (149.8, 68.5)
- moved REF** 0.13 mm to (160.0, 58.3)
- moved REF** 0.13 mm to (160.0, 65.9)
- moved REF** 0.13 mm to (149.8, 81.2)
- moved REF** 0.13 mm to (160.0, 76.1)
- moved REF** 0.13 mm to (149.8, 65.9)
- moved REF** 0.13 mm to (149.8, 86.2)
- moved REF** 0.13 mm to (149.8, 71.0)
- moved REF** 0.13 mm to (160.0, 81.2)
- moved REF** 0.13 mm to (160.0, 71.0)
- moved REF** 0.13 mm to (160.0, 68.5)
- moved REF** 0.13 mm to (160.0, 60.8)
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Other:
- board size 24.4 x 32.7 mm -> 24 x 42 mm
- board text added: "C.Brooks 2025"
- board text added: "Proto+"
- board text added: "WARNING: EXPERIMENTAL"
