File: boards/altbier-proto/AltbierProto.kicad_pcb (KiCad board)
At the start: 2 copper layers, 76.2 x 82.5 mm, 105 parts

Commit message: remove unneeded silk logo
Parts:
- removed the G*** at (141.1, 104.9)
- moved Ref** 42.0 mm to (141.2, 104.0)
