File: boards/simple-smt-proto/protoboard.kicad_sch (KiCad schematic)
At the start: 1755 parts, among them P1 PAD, P10 PAD, P11 PAD, P12 PAD, P13 PAD, P14 PAD, P15 PAD, P16 PAD, P17 PAD, P18 PAD, P19 PAD, P2 PAD, P20 PAD, P21 PAD, P22 PAD, P23 PAD, P24 PAD, P25 PAD, P26 PAD, P27 PAD, P28 PAD, P29 PAD, P3 PAD, P30 PAD, P31 PAD, P32 PAD, P33 PAD, P34 PAD, P35 PAD, P36 PAD, P37 PAD, P38 PAD, P39 PAD, P4 PAD, P40 PAD, P41 PAD, P42 PAD, P43 PAD, P44 PAD, P45 PAD, P5 PAD, P6 PAD, P7 PAD, P8 PAD, P9 PAD, U1 PROTO_SOIC6, U10 PROTO_SOT23, U100 PAD, U1000 PAD, U1001 PAD, U1002 PAD, U1003 PAD, U1004 PAD, U1005 PAD, U1006 PAD, U1007 PAD, U1008 PAD, U1009 PAD, U101 PAD, U1010 PAD, U1011 PAD, U1012 PAD, U1013 PAD, U1014 PAD, U1015 PAD, U1016 PAD, U1017 PAD, U1018 PAD, U1019 PAD, U102 PAD, U1020 PAD, U1021 PAD, U1022 PAD, U1023 PAD, U1024 PAD, U1025 PAD, U1026 PAD, U1027 PAD, U1028 PAD, U1029 PAD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

Commit message: revise smt proto
Other:
- note added: "Bottom"
- note added: "Top"
- moved on the sheet: H1, H2, H3, H4, P1, P10, P11, P12, P13, P14, P15, P16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
