File: boards/classic-protoboard_10x24/classic-protoboard_10x24.kicad_pcb (KiCad board)
At the start: 2 copper layers, 70 x 30 mm, 37 parts

Commit message: review and revise all then regen all outputs
Other:
- board text removed: "24x10 thruhole"
- board text removed: "70mm x 30mm"
- board text removed: "C.Brooks 2025"
- board text removed: "Classic Protoboard"
- board text removed: "Pitch 2.54mm"
