File: boards/classic-protoboard_14x20/classic-protoboard_14x20.kicad_pcb (KiCad board)
At the start: 2 copper layers, 60 x 40 mm, 53 parts

Commit message: review and revise all then regen all outputs
Other:
- board text removed: "20x14 thruhole"
- board text removed: "60mm x 40mm"
- board text removed: "Classic Protoboard"
- board text removed: "Pitch 2.54mm"
