File: boards/classic-protoboard_6x28/classic-protoboard_6x28.kicad_pcb (KiCad board)
At the start: 2 copper layers, 80 x 20 mm, 21 parts

Commit message: review and revise all then regen all outputs
Other:
- board text removed: "28x06 thruhole"
- board text removed: "80mm x 20mm"
- board text removed: "C.Brooks 2025"
- board text removed: "Classic Protoboard"
- board text removed: "Pitch 2.54mm"
